File: CAN-Weichendecoder_Magnet/Board/can-weichendecoder-magnet.brd (EAGLE design)
At the start: 90 x 80 mm, 36 parts, among them IC1 MCP 2562, IC2 MCP 2515, IC3 ATMEGA 328P, IC4 ULN 2803A, IC5 7805TV, Q1 16M, Q2 16M, X1 RJ45-6L21-B, X2 RJ45-6L21-B

Commit message: Kleine Änderungen und aufräumen (v0.1, Rev A)
Parts:
- added SV7: CAN, con-lstb:MA03-1
- added SV8: I²C, con-lstb:MA03-1
- moved C7 1.27 mm to (63.5, 18.4)
- moved C8 1.27 mm to (55.9, 18.4)
- moved IC5 1.27 mm to (57.1, 10.8)
- moved SV6 1.27 mm to (57.1, 5.40)
Connections:
- new net N$33: IC3.28, SV8.1
- new net N$34: IC3.27, SV8.2
- net CAN-H: now also SV7.2
- net CAN-L: now also SV7.3
- net GND: now also SV7.1, SV8.3
- net N$28: now also IC3.26; no longer IC3.28
- net N$29: now also IC3.25; no longer IC3.27
- net N$30: now also IC3.24; no longer IC3.26
- net N$31: now also IC3.23; no longer IC3.25
Routing:
- net N$34: track 0.00 -> 53.0 mm, vias 0 -> 1
- net N$33: track 0.00 -> 50.3 mm, vias 0 -> 1
- net CAN-H: track 69.0 -> 77.3 mm
- net N$31: track 55.0 -> 59.3 mm
- net N$30: track 49.4 -> 53.7 mm
- net N$29: track 43.8 -> 48.1 mm
- net N$28: track 37.7 -> 42.0 mm
- net 18V: track 130.2 -> 126.4 mm
- net CAN-L: track 69.8 -> 73.1 mm, vias 0 -> 1
- net SCK: track 38.0 -> 36.9 mm
- net VCC: track 105.7 -> 106.7 mm
Other:
- board size 90 x 80 mm -> 90 x 60 mm
- board text added: "18V"
- board text added: "5V"
- board text added: "C_H"
- board text added: "C_L"
- board text added: "MäCAN-Weichendecoder V 0.1; Rev A"
- board text removed: "+18V"
- board text removed: "+5V"
