File: CAN-Weichendecoder_Magnet/Board/can-weichendecoder-magnet.sch (EAGLE design)
At the start: 36 parts, among them IC1 MCP 2562, IC2 MCP 2515, IC3 ATMEGA 328P, IC4 ULN 2803A, IC5 7805TV, Q1 16M, Q2 16M, X1 RJ45-6L21-B, X2 RJ45-6L21-B

Commit message: Kleine Änderungen und aufräumen (v0.1, Rev A)
Parts:
- added SV7: CAN, con-lstb:MA03-1
- added SV8: I²C, con-lstb:MA03-1
Connections:
- new net N$33: IC3.28, SV8.1
- new net N$34: IC3.27, SV8.2
- net CAN-H: now also SV7.2
- net CAN-L: now also SV7.3
- net GND: now also SV7.1, SV8.3
- net N$28: now also IC3.26; no longer IC3.28
- net N$29: now also IC3.25; no longer IC3.27
- net N$30: now also IC3.24; no longer IC3.26
- net N$31: now also IC3.23; no longer IC3.25
Changed lines of the file:
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@@
 <part name="X2" library="con-tycoelectronics" deviceset="RJ45*2" device="1-B" technology="-6L"/>
 <part name="GND3" library="supply1" deviceset="GND" device=""/>
+<part name="SV7" library="con-lstb" deviceset="MA03-1" device="" value="CAN"/>
+<part name="SV8" library="con-lstb" deviceset="MA03-1" device="" value="I²C"/>
 </parts>
 <sheets>
@@
 <instance part="X2" gate="G$1" x="-15.24" y="60.96" rot="R180"/>
 <instance part="GND3" gate="1" x="210.82" y="27.94"/>
+<instance part="SV7" gate="G$1" x="-17.78" y="35.56"/>
+<instance part="SV8" gate="G$1" x="208.28" y="55.88" rot="R180"/>
 </instances>
 <busses>
@@
 </segment>
 <segment>
-<wire x1="17.78" y1="43.18" x2="15.24" y2="43.18" width="0.1524" layer="91"/>
-<label x="15.24" y="43.18" size="1.27" layer="95" rot="R180" xref="yes"/>
+<label x="12.7" y="43.18" size="1.27" layer="95" rot="R90" xref="yes"/>
 <pinref part="R3" gate="G$1" pin="2"/>
+<wire x1="17.78" y1="43.18" x2="-2.54" y2="43.18" width="0.1524" layer="91"/>
+<wire x1="-2.54" y1="43.18" x2="-2.54" y2="38.1" width="0.1524" layer="91"/>
+<pinref part="SV7" gate="G$1" pin="3"/>
+<wire x1="-2.54" y1="38.1" x2="-10.16" y2="38.1" width="0.1524" layer="91"/>
 </segment>
 </net>
@@
 <segment>
 <pinref part="JP1" gate="A" pin="2"/>
-<wire x1="27.94" y1="40.64" x2="15.24" y2="40.64" width="0.1524" layer="91"/>
-<label x="15.24" y="40.64" size="1.27" layer="95" rot="R180" xref="yes"/>
+<wire x1="27.94" y1="40.64" x2="0" y2="40.64" width="0.1524" layer="91"/>
+<label x="12.7" y="40.64" size="1.27" layer="95" rot="R270" xref="yes"/>
+<wire x1="0" y1="40.64" x2="0" y2="35.56" width="0.1524" layer="91"/>
+<pinref part="SV7" gate="G$1" pin="2"/>
+<wire x1="0" y1="35.56" x2="-10.16" y2="35.56" width="0.1524" layer="91"/>
 </segment>
 </net>
@@
 <wire x1="68.58" y1="40.64" x2="66.04" y2="40.64" width="0.1524" layer="91"/>
 <junction x="66.04" y="40.64"/>
+<pinref part="SV7" gate="G$1" pin="1"/>
+<wire x1="-10.16" y1="33.02" x2="38.1" y2="33.02" width="0.1524" layer="91"/>
+<junction x="38.1" y="33.02"/>
 </segment>
 <segment>
@@
 <pinref part="GND3" gate="1" pin="GND"/>
 <pinref part="IC3" gate="G$1" pin="22"/>
-<wire x1="185.42" y1="43.18" x2="210.82" y2="43.18" width="0.1524" layer="91"/>
+<wire x1="185.42" y1="43.18" x2="200.66" y2="43.18" width="0.1524" layer="91"/>
 <junction x="210.82" y="43.18"/>
+<pinref part="SV8" gate="G$1" pin="3"/>
+<wire x1="200.66" y1="43.18" x2="210.82" y2="43.18" width="0.1524" layer="91"/>
+<wire x1="200.66" y1="53.34" x2="200.66" y2="43.18" width="0.1524" layer="91"/>
+<junction x="200.66" y="43.18"/>
 </segment>
 </net>
@@
 <pinref part="R6" gate="G$1" pin="2"/>
 <wire x1="187.96" y1="96.52" x2="190.5" y2="96.52" width="0.1524" layer="91"/>
-<wire x1="190.5" y1="96.52" x2="190.5" y2="58.42" width="0.1524" layer="91"/>
-<pinref part="IC3" gate="G$1" pin="28"/>
-<wire x1="190.5" y1="58.42" x2="185.42" y2="58.42" width="0.1524" layer="91"/>
+<wire x1="190.5" y1="96.52" x2="190.5" y2="53.34" width="0.1524" layer="91"/>
 <pinref part="R10" gate="G$1" pin="1"/>
 <wire x1="190.5" y1="96.52" x2="200.66" y2="96.52" width="0.1524" layer="91"/>
 <junction x="190.5" y="96.52"/>
+<pinref part="IC3" gate="G$1" pin="26"/>
+<wire x1="185.42" y1="53.34" x2="190.5" y2="53.34" width="0.1524" layer="91"/>
 </segment>
 </net>
@@
 <pinref part="R7" gate="G$1" pin="2"/>
 <wire x1="187.96" y1="91.44" x2="193.04" y2="91.44" width="0.1524" layer="91"/>
-<wire x1="193.04" y1="91.44" x2="193.04" y2="55.88" width="0.1524" layer="91"/>
-<pinref part="IC3" gate="G$1" pin="27"/>
-<wire x1="193.04" y1="55.88" x2="185.42" y2="55.88" width="0.1524" layer="91"/>
+<wire x1="193.04" y1="91.44" x2="193.04" y2="50.8" width="0.1524" layer="91"/>
 <pinref part="R11" gate="G$1" pin="1"/>
 <wire x1="193.04" y1="91.44" x2="200.66" y2="91.44" width="0.1524" layer="91"/>
 <junction x="193.04" y="91.44"/>
+<pinref part="IC3" gate="G$1" pin="25"/>
+<wire x1="185.42" y1="50.8" x2="193.04" y2="50.8" width="0.1524" layer="91"/>
 </segment>
 </net>
@@
 <pinref part="R8" gate="G$1" pin="2"/>
 <wire x1="187.96" y1="86.36" x2="195.58" y2="86.36" width="0.1524" layer="91"/>
-<wire x1="195.58" y1="86.36" x2="195.58" y2="53.34" width="0.1524" layer="91"/>
-<pinref part="IC3" gate="G$1" pin="26"/>
-<wire x1="195.58" y1="53.34" x2="185.42" y2="53.34" width="0.1524" layer="91"/>
+<wire x1="195.58" y1="86.36" x2="195.58" y2="48.26" width="0.1524" layer="91"/>
 <pinref part="R12" gate="G$1" pin="1"/>
 <wire x1="195.58" y1="86.36" x2="200.66" y2="86.36" width="0.1524" layer="91"/>
 <junction x="195.58" y="86.36"/>
+<pinref part="IC3" gate="G$1" pin="24"/>
+<wire x1="185.42" y1="48.26" x2="195.58" y2="48.26" width="0.1524" layer="91"/>
 </segment>
 </net>
@@
 <pinref part="R9" gate="G$1" pin="2"/>
 <wire x1="187.96" y1="81.28" x2="198.12" y2="81.28" width="0.1524" layer="91"/>
-<wire x1="198.12" y1="81.28" x2="198.12" y2="50.8" width="0.1524" layer="91"/>
-<pinref part="IC3" gate="G$1" pin="25"/>
-<wire x1="198.12" y1="50.8" x2="185.42" y2="50.8" width="0.1524" layer="91"/>
+<wire x1="198.12" y1="81.28" x2="198.12" y2="45.72" width="0.1524" layer="91"/>
 <pinref part="R13" gate="G$1" pin="1"/>
 <wire x1="198.12" y1="81.28" x2="200.66" y2="81.28" width="0.1524" layer="91"/>
 <junction x="198.12" y="81.28"/>
+<pinref part="IC3" gate="G$1" pin="23"/>
+<wire x1="185.42" y1="45.72" x2="198.12" y2="45.72" width="0.1524" layer="91"/>
 </segment>
 </net>
@@
 </segment>
 </net>
+<net name="N$33" class="0">
+<segment>
+<pinref part="SV8" gate="G$1" pin="1"/>
+<pinref part="IC3" gate="G$1" pin="28"/>
+<wire x1="200.66" y1="58.42" x2="185.42" y2="58.42" width="0.1524" layer="91"/>
+</segment>
+</net>
+<net name="N$34" class="0">
+<segment>
+<pinref part="IC3" gate="G$1" pin="27"/>
+<pinref part="SV8" gate="G$1" pin="2"/>
+<wire x1="185.42" y1="55.88" x2="200.66" y2="55.88" width="0.1524" layer="91"/>
+</segment>
+</net>
