File: CAN-Weichendecoder_Magnet/Board/Eagle/can-weichendecoder-magnet.brd (EAGLE design)
At the start: 90 x 60 mm, 38 parts, among them IC1 MCP 2562, IC2 MCP 2515, IC3 ATMEGA 328P, IC4 ULN 2803A, IC5 7805TV, Q1 16M, Q2 16M

Commit message: Added files via upload
Parts:
- SV8: value I²C -> (none); device con-lstb:MA03-1 -> con-lstb:MA04-1
- moved SV8 1.79 mm to (86.4, 31.8)
Connections:
- net VCC: now also SV8.4
Routing:
- net VCC: track 108.0 -> 157.0 mm
- net N$34: track 53.0 -> 53.5 mm
Changed lines of the file:
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@@
 <wire x1="2.5" y1="0" x2="0" y2="2.5" width="0" layer="20" curve="-90"/>
 <wire x1="0" y1="2.5" x2="0" y2="57.5" width="0" layer="20"/>
-<dimension x1="87" y1="3" x2="87" y2="57" x3="96" y3="30" textsize="1.778" layer="27" dtype="vertical"/>
-<dimension x1="87" y1="3" x2="3" y2="3" x3="45" y3="-7" textsize="1.778" layer="27" dtype="horizontal"/>
-<dimension x1="0" y1="2.5" x2="90" y2="2.5" x3="45" y3="-10" textsize="1.778" layer="27" dtype="horizontal"/>
-<dimension x1="87.5" y1="0" x2="87" y2="60" x3="99" y3="30" textsize="1.778" layer="27" dtype="vertical"/>
-<dimension x1="4.6" y1="3" x2="1.4" y2="3" x3="3" y3="-6" textsize="1.778" layer="27" dtype="diameter"/>
 <text x="6.985" y="25.4" size="1.778" layer="21" rot="R180">.</text>
 </plain>
@@
 <attribute name="MF" value="" x="47.625" y="5.3975" size="1.778" layer="27" display="off"/>
 </element>
-<element name="SV8" library="con-lstb" package="MA03-1" value="I²C" x="86" y="30" rot="R90">
-<attribute name="MF" value="" x="86" y="30" size="1.778" layer="27" rot="R90" display="off"/>
-<attribute name="MPN" value="" x="86" y="30" size="1.778" layer="27" rot="R90" display="off"/>
-<attribute name="OC_NEWARK" value="unknown" x="86" y="30" size="1.778" layer="27" rot="R90" display="off"/>
-<attribute name="OC_FARNELL" value="unknown" x="86" y="30" size="1.778" layer="27" rot="R90" display="off"/>
-</element>
 <element name="J1" library="con-amp" package="215877-7" value="" x="15" y="5"/>
 <element name="J2" library="con-amp" package="215877-7" value="" x="75" y="5"/>
 <element name="C7" library="rcl" package="E2,5-6" value="0,1µ" x="60.96" y="12.7" smashed="yes">
 <attribute name="NAME" x="63.627" y="14.224" size="1.27" layer="25" ratio="10"/>
+</element>
+<element name="SV8" library="con-lstb" package="MA04-1" value="" x="86.36" y="31.75" rot="R90">
+<attribute name="OC_FARNELL" value="unknown" x="86.36" y="31.75" size="1.778" layer="27" rot="R90" display="off"/>
+<attribute name="MF" value="" x="86.36" y="31.75" size="1.778" layer="27" rot="R90" display="off"/>
+<attribute name="OC_NEWARK" value="unknown" x="86.36" y="31.75" size="1.778" layer="27" rot="R90" display="off"/>
+<attribute name="MPN" value="" x="86.36" y="31.75" size="1.778" layer="27" rot="R90" display="off"/>
 </element>
 </elements>
@@
 <wire x1="54.61" y1="12.7" x2="54.61" y2="5.3975" width="1.27" layer="16"/>
 <wire x1="54.61" y1="15.24" x2="35.56" y2="15.24" width="0.6096" layer="16"/>
+<contactref element="SV8" pad="4"/>
+<wire x1="86.36" y1="35.56" x2="87.63" y2="35.56" width="0.8128" layer="1"/>
+<wire x1="87.63" y1="35.56" x2="88.9" y2="34.29" width="0.8128" layer="1"/>
+<wire x1="88.9" y1="34.29" x2="88.9" y2="26.67" width="0.8128" layer="1"/>
+<wire x1="88.9" y1="26.67" x2="87.63" y2="25.4" width="0.8128" layer="1"/>
+<wire x1="87.63" y1="25.4" x2="82.55" y2="25.4" width="0.8128" layer="1"/>
+<wire x1="82.55" y1="25.4" x2="81.28" y2="24.13" width="0.8128" layer="1"/>
+<wire x1="81.28" y1="24.13" x2="57.15" y2="24.13" width="0.8128" layer="1"/>
+<wire x1="57.15" y1="24.13" x2="54.61" y2="21.59" width="0.8128" layer="1"/>
+<wire x1="54.61" y1="21.59" x2="54.61" y2="19.685" width="0.8128" layer="1"/>
 </signal>
 <signal name="N$9">
@@
 <contactref element="C4" pad="1"/>
 <contactref element="SV7" pad="1"/>
-<contactref element="SV8" pad="3"/>
 <contactref element="J1" pad="3"/>
 <contactref element="J1" pad="4"/>
@@
 <vertex x="-1.27" y="60.96"/>
 </polygon>
+<contactref element="SV8" pad="3"/>
 </signal>
 <signal name="RESET">
@@
 </signal>
 <signal name="N$33">
-<contactref element="SV8" pad="1"/>
 <contactref element="IC3" pad="28"/>
 <wire x1="40.64" y1="38.1" x2="46.355" y2="32.385" width="0.4064" layer="16"/>
@@
 <wire x1="46.99" y1="33.02" x2="68.58" y2="33.02" width="0.4064" layer="1"/>
 <wire x1="68.58" y1="33.02" x2="73.66" y2="27.94" width="0.4064" layer="1"/>
-<wire x1="73.66" y1="27.94" x2="85.52" y2="27.94" width="0.4064" layer="1"/>
-<wire x1="85.52" y1="27.94" x2="86" y2="27.46" width="0.4064" layer="1"/>
+<wire x1="73.66" y1="27.94" x2="86.36" y2="27.94" width="0.4064" layer="1"/>
+<contactref element="SV8" pad="1"/>
 </signal>
 <signal name="N$34">
 <contactref element="IC3" pad="27"/>
-<contactref element="SV8" pad="2"/>
-<wire x1="84.575" y1="28.575" x2="74.295" y2="28.575" width="0.4064" layer="1"/>
 <wire x1="74.295" y1="28.575" x2="69.215" y2="33.655" width="0.4064" layer="1"/>
 <wire x1="69.215" y1="33.655" x2="43.815" y2="33.655" width="0.4064" layer="1"/>
@@
 <via x="43.18" y="33.02" extent="1-16" drill="0.6"/>
 <wire x1="43.18" y1="33.02" x2="38.1" y2="38.1" width="0.4064" layer="16"/>
-<wire x1="84.575" y1="28.575" x2="86" y2="30" width="0.4064" layer="1"/>
+<contactref element="SV8" pad="2"/>
+<wire x1="74.295" y1="28.575" x2="84.455" y2="28.575" width="0.4064" layer="1"/>
+<wire x1="84.455" y1="28.575" x2="86.36" y2="30.48" width="0.4064" layer="1"/>
 </signal>
 </signals>
