File: CAN-Weichendecoder_Magnet/Board/Eagle/can-weichendecoder-magnet.sch (EAGLE design)
At the start: 38 parts, among them IC1 MCP 2562, IC2 MCP 2515, IC3 ATMEGA 328P, IC4 ULN 2803A, IC5 7805TV, Q1 16M, Q2 16M

Commit message: Added files via upload
Parts:
- SV8: value I²C -> (none); device con-lstb:MA03-1 -> con-lstb:MA04-1
Connections:
- net VCC: now also SV8.4
Changed lines of the file:
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@@
 <part name="GND3" library="supply1" deviceset="GND" device=""/>
 <part name="SV7" library="con-lstb" deviceset="MA03-1" device="" value="CAN"/>
-<part name="SV8" library="con-lstb" deviceset="MA03-1" device="" value="I²C"/>
 <part name="J1" library="con-amp" deviceset="215877-7" device=""/>
 <part name="J2" library="con-amp" deviceset="215877-7" device=""/>
 <part name="C7" library="rcl" deviceset="CPOL-EU" device="E2.5-6" value="0,1µ"/>
+<part name="SV8" library="con-lstb" deviceset="MA04-1" device=""/>
 </parts>
 <sheets>
@@
 <instance part="GND3" gate="1" x="210.82" y="27.94"/>
 <instance part="SV7" gate="G$1" x="-17.78" y="35.56"/>
-<instance part="SV8" gate="G$1" x="208.28" y="55.88" rot="R180"/>
 <instance part="J1" gate="G$1" x="-12.7" y="86.36" rot="R180"/>
 <instance part="J2" gate="G$1" x="-12.7" y="58.42" rot="R180"/>
 <instance part="C7" gate="G$1" x="48.26" y="104.14"/>
+<instance part="SV8" gate="1" x="223.52" y="53.34" rot="R180"/>
 </instances>
 <busses>
@@
 <segment>
 <pinref part="IC3" gate="G$1" pin="20"/>
-<wire x1="185.42" y1="38.1" x2="187.96" y2="38.1" width="0.1524" layer="91"/>
 <pinref part="IC3" gate="G$1" pin="21"/>
-<wire x1="185.42" y1="40.64" x2="187.96" y2="38.1" width="0.1524" layer="91"/>
-<label x="187.96" y="38.1" size="1.27" layer="95" xref="yes"/>
+<wire x1="185.42" y1="40.64" x2="185.42" y2="38.1" width="0.1524" layer="91"/>
+<label x="185.42" y="38.1" size="1.27" layer="95" xref="yes"/>
+<pinref part="SV8" gate="1" pin="4"/>
+<wire x1="215.9" y1="50.8" x2="215.9" y2="40.64" width="0.1524" layer="91"/>
+<wire x1="215.9" y1="40.64" x2="185.42" y2="40.64" width="0.1524" layer="91"/>
+<junction x="185.42" y="40.64"/>
 </segment>
 <segment>
@@
 <pinref part="IC4" gate="G$1" pin="9"/>
 <wire x1="165.1" y1="63.5" x2="210.82" y2="63.5" width="0.1524" layer="91"/>
-<wire x1="210.82" y1="63.5" x2="210.82" y2="43.18" width="0.1524" layer="91"/>
+<wire x1="210.82" y1="63.5" x2="210.82" y2="53.34" width="0.1524" layer="91"/>
+<wire x1="210.82" y1="53.34" x2="210.82" y2="43.18" width="0.1524" layer="91"/>
 <wire x1="210.82" y1="43.18" x2="210.82" y2="30.48" width="0.1524" layer="91"/>
 <wire x1="210.82" y1="81.28" x2="210.82" y2="63.5" width="0.1524" layer="91"/>
@@
 <pinref part="GND3" gate="1" pin="GND"/>
 <pinref part="IC3" gate="G$1" pin="22"/>
-<wire x1="185.42" y1="43.18" x2="200.66" y2="43.18" width="0.1524" layer="91"/>
+<wire x1="185.42" y1="43.18" x2="210.82" y2="43.18" width="0.1524" layer="91"/>
 <junction x="210.82" y="43.18"/>
-<pinref part="SV8" gate="G$1" pin="3"/>
-<wire x1="200.66" y1="43.18" x2="210.82" y2="43.18" width="0.1524" layer="91"/>
-<wire x1="200.66" y1="53.34" x2="200.66" y2="43.18" width="0.1524" layer="91"/>
-<junction x="200.66" y="43.18"/>
+<pinref part="SV8" gate="1" pin="3"/>
+<wire x1="215.9" y1="53.34" x2="210.82" y2="53.34" width="0.1524" layer="91"/>
+<junction x="210.82" y="53.34"/>
 </segment>
 </net>
@@
 <net name="N$33" class="0">
 <segment>
-<pinref part="SV8" gate="G$1" pin="1"/>
 <pinref part="IC3" gate="G$1" pin="28"/>
-<wire x1="200.66" y1="58.42" x2="185.42" y2="58.42" width="0.1524" layer="91"/>
+<pinref part="SV8" gate="1" pin="1"/>
+<wire x1="185.42" y1="58.42" x2="215.9" y2="58.42" width="0.1524" layer="91"/>
 </segment>
 </net>
@@
 <segment>
 <pinref part="IC3" gate="G$1" pin="27"/>
-<pinref part="SV8" gate="G$1" pin="2"/>
-<wire x1="185.42" y1="55.88" x2="200.66" y2="55.88" width="0.1524" layer="91"/>
-</segment>
-</net>
+<pinref part="SV8" gate="1" pin="2"/>
+<wire x1="185.42" y1="55.88" x2="215.9" y2="55.88" width="0.1524" layer="91"/>
+</segment>
+</net>
