File: CAN-UDP-Bridge/board/Eagle/can-udp-bridge.pan.brd (EAGLE design)
At the start: 23.8 x 35.5 mm, 15 parts, among them IC2 MCP1703DB, Q1 16M, X1 B4B-ZR

Commit message: Added files via upload
Parts:
- added C10, C9: 1µ, rcl:C0805
- added C4, C7: 22p, rcl:C0805
- added C8: 100n, rcl:C0805
- added CAN-TERM1: (no value), jumper:SJ
- added IC1: MCP1703DB, linear:SOT223
- added MDL2: (no value), ESP8266-ESP12E:ESP8266-ESP12E
- added PROG1: (no value), con-lsta:FE06W
- added Q2: 16M, crystal:CTS406
- added R1: 120R, rcl:R0805
- added U$4: MCP2515-I/SO, Microchip_By_element14_Batch_1:SOIC127P1034X264-18N
- added U$5: MCP2551-E/SN, Microchip_By_element14_Batch_1:SOIC127P600X175-8N
- added U$6: ROF-78E5.0-0.5SMD, ROF-78XX:ROF-78EXX-0.5SMD
- added X2: B4B-ZR, con-jst:B4B-ZR
Connections:
- new net +18V1: U$6.1, X2.1
- new net +3V1: C8.1, C9.2, IC1.3, MDL2.8, PROG1.4, U$4.18, U$5.5
- new net +5V1: C10.2, IC1.1, U$5.3, U$6.3
- new net CAN_H1: CAN-TERM1.1, U$5.7, X2.2
- new net CAN_L1: R1.1, U$5.6, X2.3
- new net GND1: C10.1, C4.2, C7.2, C8.2, C9.1, IC1.2, MDL2.9, PROG1.6, U$4.9, U$5.2, U$5.8, U$6.2, X2.4
- new net N$12: U$4.1, U$5.1
- new net N$16: U$4.2, U$5.4
- new net N$17: MDL2.16, PROG1.1
- new net N$18: MDL2.15, PROG1.2
- new net N$19: MDL2.18, U$4.15
- new net N$20: MDL2.10, U$4.16
- new net N$21: MDL2.21, U$4.14
- new net N$22: MDL2.11, U$4.12
- new net N$23: MDL2.22, U$4.13
- new net N$24: MDL2.1, PROG1.3
- new net N$25: MDL2.12, PROG1.5
- new net N$26: C4.1, Q2.3, U$4.7
- new net N$27: C7.1, Q2.1, U$4.8
- new net N$28: CAN-TERM1.2, R1.2
Routing:
- net +3V1: track 0.00 -> 53.8 mm, vias 0 -> 3
- net N$24: track 0.00 -> 31.7 mm, vias 0 -> 1
- net CAN_L1: track 0.00 -> 27.9 mm, vias 0 -> 1
- net N$17: track 0.00 -> 26.6 mm
- net N$18: track 0.00 -> 25.7 mm
- net CAN_H1: track 0.00 -> 23.5 mm, vias 0 -> 1
- net +18V1: track 0.00 -> 21.0 mm
- net N$25: track 0.00 -> 17.3 mm, vias 0 -> 2
- net +5V1: track 0.00 -> 14.8 mm
- net N$20: track 0.00 -> 14.6 mm, vias 0 -> 1
- net N$27: track 0.00 -> 11.9 mm
- net N$26: track 0.00 -> 10.8 mm
- net N$22: track 0.00 -> 10.5 mm, vias 0 -> 1
- net N$12: track 0.00 -> 9.79 mm
- net N$19: track 0.00 -> 7.64 mm, vias 0 -> 1
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- added copper zone on layer 1, net GND1
- added copper zone on layer 16, net GND1
Other:
- board size 23.8 x 35.5 mm -> 48.9 x 35.6 mm
