File: CAN-UDP-Bridge/board/Eagle/can-udp-bridge_0_2.pan.brd (EAGLE design)
At the start: 99.1 x 63.2 mm, 92 parts, among them IC1 MCP1703DB, IC2 MCP1703DB, IC3 MCP1703DB, IC4 MCP1703DB, Q1 16M, Q2 16M, Q3 16M, Q4 16M, X1 B4B-ZR, X2 B4B-ZR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

Commit message: Anpassungen
Changed lines of the file:
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@@
 <plain>
 <wire x1="2.54" y1="0" x2="21.2725" y2="0" width="0" layer="20"/>
-<text x="7.14375" y="5.08" size="1.016" layer="25" rot="R90">0</text>
-<text x="8.73125" y="5.08" size="1.016" layer="25">GND</text>
-<text x="17.30375" y="5.08" size="1.016" layer="25" rot="R90">TX</text>
-<text x="14.76375" y="5.08" size="1.016" layer="25" rot="R90">RX</text>
+<text x="7.14375" y="5.08" size="1.016" layer="125" rot="R90">0</text>
+<text x="8.73125" y="5.08" size="1.016" layer="125">GND</text>
+<text x="17.30375" y="5.08" size="1.016" layer="125" rot="R90">TX</text>
+<text x="14.76375" y="5.08" size="1.016" layer="125" rot="R90">RX</text>
 <wire x1="0" y1="35.8775" x2="0" y2="2.54" width="0" layer="20"/>
 <wire x1="0" y1="60.6425" x2="0" y2="41.91" width="0" layer="20"/>
@@
 <dimension x1="26.3525" y1="73.66" x2="26.3525" y2="10.4775" x3="-8.5725" y3="42.06875" textsize="1.778" layer="47" dtype="vertical"/>
 <dimension x1="5.08" y1="71.12" x2="28.8925" y2="71.12" x3="16.98625" y3="80.645" textsize="1.778" layer="47" dtype="vertical"/>
-<text x="19.3675" y="44.1325" size="1.778" layer="25">r</text>
-<text x="12.3825" y="44.1325" size="1.778" layer="25">b</text>
+<text x="19.3675" y="44.1325" size="1.778" layer="125">r</text>
+<text x="12.3825" y="44.1325" size="1.778" layer="125">b</text>
 <wire x1="0" y1="2.54" x2="2.54" y2="5.08" width="0" layer="21" curve="-90"/>
 <wire x1="2.54" y1="5.08" x2="5.08" y2="2.54" width="0" layer="21" curve="-90"/>
@@
 <text x="12.780009375" y="8.349996875" size="1.27" layer="122" rot="MR90">MDL1</text>
 <text x="1.905" y="12.7" size="1.27" layer="125">Q1</text>
-<text x="3.81" y="9.525" size="1.27" layer="125" rot="R180">R1</text>
+<text x="4.7625" y="6.0325" size="1.27" layer="125" rot="R180">R1</text>
 <text x="20.6375" y="9.8425" size="1.27" layer="126" rot="MR180">R2</text>
 <text x="18.415" y="8.255" size="1.27" layer="125">R4</text>
 <wire x1="27.6225" y1="0" x2="46.355" y2="0" width="0" layer="20"/>
-<text x="32.22625" y="5.08" size="1.016" layer="25" rot="R90">0</text>
-<text x="33.81375" y="5.08" size="1.016" layer="25">GND</text>
-<text x="42.38625" y="5.08" size="1.016" layer="25" rot="R90">TX</text>
-<text x="39.84625" y="5.08" size="1.016" layer="25" rot="R90">RX</text>
+<text x="32.22625" y="5.08" size="1.016" layer="125" rot="R90">0</text>
+<text x="33.81375" y="5.08" size="1.016" layer="125">GND</text>
+<text x="42.38625" y="5.08" size="1.016" layer="125" rot="R90">TX</text>
+<text x="39.84625" y="5.08" size="1.016" layer="125" rot="R90">RX</text>
 <wire x1="25.0825" y1="60.6425" x2="25.0825" y2="54.9275" width="0" layer="20"/>
 <text x="41.275" y="48.26" size="1.016" layer="16" font="vector" ratio="15" rot="MR90">MäCAN Adap
@@
 <wire x1="46.355" y1="38.4175" x2="48.895" y2="35.8775" width="0" layer="20" curve="-90"/>
 <wire x1="25.0825" y1="35.8775" x2="27.6225" y2="38.4175" width="0" layer="20" curve="-90"/>
-<text x="44.45" y="44.1325" size="1.778" layer="25">r</text>
-<text x="37.465" y="44.1325" size="1.778" layer="25">b</text>
+<text x="44.45" y="44.1325" size="1.778" layer="125">r</text>
+<text x="37.465" y="44.1325" size="1.778" layer="125">b</text>
 <wire x1="25.0825" y1="2.54" x2="27.6225" y2="5.08" width="0" layer="21" curve="-90"/>
 <wire x1="27.6225" y1="5.08" x2="30.1625" y2="2.54" width="0" layer="21" curve="-90"/>
@@
 <text x="37.862509375" y="8.349996875" size="1.27" layer="122" rot="MR90">MDL1</text>
 <text x="26.9875" y="12.7" size="1.27" layer="125">Q1</text>
-<text x="28.8925" y="9.525" size="1.27" layer="125" rot="R180">R1</text>
+<text x="29.845" y="6.0325" size="1.27" layer="125" rot="R180">R1</text>
 <text x="45.72" y="9.8425" size="1.27" layer="126" rot="MR180">R2</text>
 <text x="43.4975" y="8.255" size="1.27" layer="125">R4</text>
 <wire x1="52.705" y1="0" x2="71.4375" y2="0" width="0" layer="20"/>
-<text x="57.30875" y="5.08" size="1.016" layer="25" rot="R90">0</text>
-<text x="58.89625" y="5.08" size="1.016" layer="25">GND</text>
-<text x="67.46875" y="5.08" size="1.016" layer="25" rot="R90">TX</text>
-<text x="64.92875" y="5.08" size="1.016" layer="25" rot="R90">RX</text>
+<text x="57.30875" y="5.08" size="1.016" layer="125" rot="R90">0</text>
+<text x="58.89625" y="5.08" size="1.016" layer="125">GND</text>
+<text x="67.46875" y="5.08" size="1.016" layer="125" rot="R90">TX</text>
+<text x="64.92875" y="5.08" size="1.016" layer="125" rot="R90">RX</text>
 <text x="66.3575" y="48.26" size="1.016" layer="16" font="vector" ratio="15" rot="MR90">MäCAN Adap
 Rev A v0.1</text>
@@
 <wire x1="71.4375" y1="38.4175" x2="73.9775" y2="35.8775" width="0" layer="20" curve="-90"/>
 <wire x1="50.165" y1="35.8775" x2="52.705" y2="38.4175" width="0" layer="20" curve="-90"/>
-<text x="69.5325" y="44.1325" size="1.778" layer="25">r</text>
-<text x="62.5475" y="44.1325" size="1.778" layer="25">b</text>
+<text x="69.5325" y="44.1325" size="1.778" layer="125">r</text>
+<text x="62.5475" y="44.1325" size="1.778" layer="125">b</text>
 <wire x1="50.165" y1="2.54" x2="52.705" y2="5.08" width="0" layer="21" curve="-90"/>
 <wire x1="52.705" y1="5.08" x2="55.245" y2="2.54" width="0" layer="21" curve="-90"/>
@@
 <text x="62.945009375" y="8.349996875" size="1.27" layer="122" rot="MR90">MDL1</text>
 <text x="52.07" y="12.7" size="1.27" layer="125">Q1</text>
-<text x="53.975" y="9.525" size="1.27" layer="125" rot="R180">R1</text>
+<text x="54.9275" y="6.0325" size="1.27" layer="125" rot="R180">R1</text>
 <text x="70.8025" y="9.8425" size="1.27" layer="126" rot="MR180">R2</text>
 <text x="68.58" y="8.255" size="1.27" layer="125">R4</text>
 <wire x1="77.7875" y1="0" x2="96.52" y2="0" width="0" layer="20"/>
-<text x="82.39125" y="5.08" size="1.016" layer="25" rot="R90">0</text>
-<text x="83.97875" y="5.08" size="1.016" layer="25">GND</text>
-<text x="92.55125" y="5.08" size="1.016" layer="25" rot="R90">TX</text>
-<text x="90.01125" y="5.08" size="1.016" layer="25" rot="R90">RX</text>
+<text x="82.39125" y="5.08" size="1.016" layer="125" rot="R90">0</text>
+<text x="83.97875" y="5.08" size="1.016" layer="125">GND</text>
+<text x="92.55125" y="5.08" size="1.016" layer="125" rot="R90">TX</text>
+<text x="90.01125" y="5.08" size="1.016" layer="125" rot="R90">RX</text>
 <text x="91.44" y="48.26" size="1.016" layer="16" font="vector" ratio="15" rot="MR90">MäCAN Adap
 Rev A v0.1</text>
@@
 <wire x1="99.06" y1="2.54" x2="99.06" y2="35.8775" width="0" layer="20"/>
 <wire x1="75.2475" y1="35.8775" x2="77.7875" y2="38.4175" width="0" layer="20" curve="-90"/>
-<text x="94.615" y="44.1325" size="1.778" layer="25">r</text>
-<text x="87.63" y="44.1325" size="1.778" layer="25">b</text>
+<text x="94.615" y="44.1325" size="1.778" layer="125">r</text>
+<text x="87.63" y="44.1325" size="1.778" layer="125">b</text>
 <wire x1="75.2475" y1="2.54" x2="77.7875" y2="5.08" width="0" layer="21" curve="-90"/>
 <wire x1="77.7875" y1="5.08" x2="80.3275" y2="2.54" width="0" layer="21" curve="-90"/>
@@
 <text x="88.027509375" y="8.349996875" size="1.27" layer="122" rot="MR90">MDL1</text>
 <text x="77.1525" y="12.7" size="1.27" layer="125">Q1</text>
-<text x="79.0575" y="9.525" size="1.27" layer="125" rot="R180">R1</text>
+<text x="80.01" y="6.0325" size="1.27" layer="125" rot="R180">R1</text>
 <text x="95.885" y="9.8425" size="1.27" layer="126" rot="MR180">R2</text>
 <text x="93.6625" y="8.255" size="1.27" layer="125">R4</text>
@@
 </element>
 <element name="R1" library="rcl" package="R0805" value="12k" x="2.8575" y="6.985" smashed="yes" rot="R180">
-<attribute name="NAME" x="3.81" y="9.525" size="1.27" layer="25" rot="R180"/>
+<attribute name="NAME" x="4.7625" y="6.0325" size="1.27" layer="25" rot="R180"/>
 </element>
 <element name="C8" library="rcl" package="C0805" value="22p" x="27.94" y="9.2075" smashed="yes" rot="R180">
