File: CAN-Universalmodul/Board/Eagle/can-universalmodul_1_0.sch (EAGLE design)
At the start: 50 parts, among them IC1 MCP 2562, IC2 MCP 2515, IC3 ATMEGA 328P, Q1 16M, Q2 16M, X1 MINI-USB-UX60-MB-5ST

Commit message: Stecker hinzugefügt
Parts:
- added X4: B4B-ZR, con-jst:B4B-ZR
Connections:
- net N$15: now also X4-3.1
- net N$16: now also X4-2.1
- net _18V: now also X4-1.1
- net _GND: now also X4-4.1
Changed lines of the file:
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@@
 <part name="JP3" library="jumper" deviceset="JP1E" device=""/>
 <part name="JP4" library="jumper" deviceset="JP1E" device=""/>
+<part name="X4" library="con-jst" deviceset="?4B-ZR" device="B"/>
 </parts>
 <sheets>
@@
 <instance part="JP3" gate="A" x="332.74" y="76.2" rot="R270"/>
 <instance part="JP4" gate="A" x="332.74" y="50.8" rot="R270"/>
+<instance part="X4" gate="-1" x="353.06" y="25.4"/>
+<instance part="X4" gate="-2" x="353.06" y="22.86"/>
+<instance part="X4" gate="-3" x="353.06" y="20.32"/>
+<instance part="X4" gate="-4" x="353.06" y="17.78"/>
 </instances>
 <busses>
@@
 <wire x1="309.88" y1="15.24" x2="312.42" y2="15.24" width="0.1524" layer="91"/>
 <junction x="312.42" y="15.24"/>
+<pinref part="X4" gate="-4" pin="1"/>
+<wire x1="347.98" y1="17.78" x2="327.66" y2="17.78" width="0.1524" layer="91"/>
+<wire x1="327.66" y1="17.78" x2="327.66" y2="15.24" width="0.1524" layer="91"/>
+<wire x1="327.66" y1="15.24" x2="312.42" y2="15.24" width="0.1524" layer="91"/>
 </segment>
 </net>
@@
 <pinref part="SV5" gate="1" pin="5"/>
 <wire x1="320.04" y1="25.4" x2="309.88" y2="25.4" width="0.1524" layer="91"/>
+<pinref part="X4" gate="-3" pin="1"/>
+<wire x1="347.98" y1="20.32" x2="320.04" y2="20.32" width="0.1524" layer="91"/>
+<wire x1="320.04" y1="20.32" x2="320.04" y2="25.4" width="0.1524" layer="91"/>
+<junction x="320.04" y="25.4"/>
 </segment>
 </net>
@@
 <wire x1="322.58" y1="27.94" x2="322.58" y2="55.88" width="0.1524" layer="91"/>
 <junction x="322.58" y="55.88"/>
+<pinref part="X4" gate="-2" pin="1"/>
+<wire x1="347.98" y1="22.86" x2="322.58" y2="22.86" width="0.1524" layer="91"/>
+<wire x1="322.58" y1="22.86" x2="322.58" y2="27.94" width="0.1524" layer="91"/>
+<junction x="322.58" y="27.94"/>
 </segment>
 </net>
@@
 <pinref part="SV5" gate="1" pin="2"/>
 <wire x1="325.12" y1="73.66" x2="325.12" y2="48.26" width="0.1524" layer="91"/>
-<wire x1="325.12" y1="48.26" x2="325.12" y2="17.78" width="0.1524" layer="91"/>
+<wire x1="325.12" y1="48.26" x2="325.12" y2="25.4" width="0.1524" layer="91"/>
+<wire x1="325.12" y1="25.4" x2="325.12" y2="17.78" width="0.1524" layer="91"/>
 <wire x1="325.12" y1="17.78" x2="325.12" y2="2.54" width="0.1524" layer="91"/>
 <wire x1="309.88" y1="17.78" x2="325.12" y2="17.78" width="0.1524" layer="91"/>
@@
 <wire x1="330.2" y1="48.26" x2="325.12" y2="48.26" width="0.1524" layer="91"/>
 <junction x="325.12" y="48.26"/>
-</segment>
-</net>
+<pinref part="X4" gate="-1" pin="1"/>
+<wire x1="347.98" y1="25.4" x2="325.12" y2="25.4" width="0.1524" layer="91"/>
+<junction x="325.12" y="25.4"/>
+</segment>
+</net>

Commit message: Anpassungen
Parts:
- added SV3: Serial, con-lstb:MA04-1
Connections:
- net 7: now also SV3.3
- net 8: now also SV3.2
- net GND: now also SV3.4
- net RESET: now also SV3.1
Changed lines of the file:
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@@
 <part name="JP4" library="jumper" deviceset="JP1E" device=""/>
 <part name="X4" library="con-jst" deviceset="?4B-ZR" device="B"/>
+<part name="SV3" library="con-lstb" deviceset="MA04-1" device="" value="Serial"/>
 </parts>
 <sheets>
@@
 <instance part="X4" gate="-3" x="353.06" y="20.32"/>
 <instance part="X4" gate="-4" x="353.06" y="17.78"/>
+<instance part="SV3" gate="1" x="251.46" y="53.34" rot="R180"/>
 </instances>
 <busses>
@@
 <pinref part="GND6" gate="1" pin="GND"/>
 </segment>
+<segment>
+<pinref part="SV3" gate="1" pin="4"/>
+<wire x1="243.84" y1="50.8" x2="241.3" y2="50.8" width="0.1524" layer="91"/>
+<label x="241.3" y="50.8" size="1.27" layer="95" rot="R180" xref="yes"/>
+</segment>
 </net>
 <net name="RESET" class="0">
@@
 <label x="12.7" y="20.32" size="1.27" layer="95" rot="R180" xref="yes"/>
 </segment>
+<segment>
+<pinref part="SV3" gate="1" pin="1"/>
+<wire x1="243.84" y1="58.42" x2="241.3" y2="58.42" width="0.1524" layer="91"/>
+<label x="241.3" y="58.42" size="1.27" layer="95" rot="R180" xref="yes"/>
+</segment>
 </net>
 <net name="CS" class="0">
@@
 <pinref part="SV4" gate="G$1" pin="3"/>
 </segment>
+<segment>
+<pinref part="SV3" gate="1" pin="2"/>
+<wire x1="243.84" y1="55.88" x2="241.3" y2="55.88" width="0.1524" layer="91"/>
+<label x="241.3" y="55.88" size="1.27" layer="95" rot="R180" xref="yes"/>
+</segment>
 </net>
 <net name="7" class="0">
@@
 <pinref part="SV4" gate="G$1" pin="4"/>
 </segment>
-</net>
+<segment>
+<pinref part="SV3" gate="1" pin="3"/>
+<wire x1="243.84" y1="53.34" x2="241.3" y2="53.34" width="0.1524" layer="91"/>
+<label x="241.3" y="53.34" size="1.27" layer="95" rot="R180" xref="yes"/>
+</segment>
+</net>

Commit message: PCB-Production-Ready
Parts:
- removed R10, R11, R12, R13, R14, R5, R6, R7, R8, R9: 10k, rcl:R-EU_R0805
- removed SV3: Serial, con-lstb:MA04-1
- added C7: 100n, rcl:C-EUC0805K
- added J6: FTDI_BASICPTH, SparkFun-Connectors:FTDI_BASICPTH
Connections:
- new net N$17: C7.2, J6.1
- net 1: no longer R5.1
- net 10: no longer R14.1
- net 2: no longer R6.1
- net 3: no longer R7.1
- net 4: no longer R8.1
- net 5: no longer R9.1
- net 6: no longer R10.1
- net 7: now also J6.2; no longer R11.1, SV3.3
- net 8: now also J6.3; no longer R12.1, SV3.2
- net 9: no longer R13.1
- net GND: now also J6.6; no longer SV3.4
- net RESET: now also C7.1; no longer SV3.1
- net VCC: no longer R10.2, R11.2, R12.2, R13.2, R14.2, R5.2, R6.2, R7.2, R8.2, R9.2
